File: hardware/project-x.sch (KiCad schematic (older format))
At the start: 23 parts, among them J1 Conn_01x02, J2 Conn_01x02, J3 Serial, J4 I2C, J5 Conn_01x02, J6 SoftSerial, J7 Conn_01x06, J8 Conn_01x02, SW1 SW_DPST, U1 TSOP382xx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

Commit message: Start basic layout
Parts:
- D1, D2, D3: footprint (none) -> LEDs:LED_0805_HandSoldering
- J1, J2, J5, J8: footprint (none) -> Pin_Headers:Pin_Header_Straight_1x02_Pitch2.54mm
- J3, J4, J6: footprint (none) -> Pin_Headers:Pin_Header_Straight_1x04_Pitch2.54mm
- J7: footprint (none) -> Pin_Headers:Pin_Header_Straight_1x06_Pitch2.54mm
- JP1: footprint (none) -> def-footprints:Miscellaneous_Solder_Jumper
- R1, R2, R3, R4, R5, R6: footprint (none) -> Resistors_SMD:R_0805_HandSoldering
- SW1: footprint (none) -> def-footprints:Switches_Push_Switch_THD
Changed lines of the file:
@@
 F 0 "J1" H 1500 4100 50  0000 C CNN
 F 1 "Conn_01x02" H 1500 3800 50  0000 C CNN
-F 2 "" H 1500 4000 50  0001 C CNN
+F 2 "Pin_Headers:Pin_Header_Straight_1x02_Pitch2.54mm" H 1500 4000 50  0001 C CNN
 F 3 "" H 1500 4000 50  0001 C CNN
 	1    1500 4000
@@
 F 0 "D1" H 6600 1300 50  0000 C CNN
 F 1 "LED" H 6600 1100 50  0000 C CNN
-F 2 "" H 6600 1200 50  0001 C CNN
+F 2 "LEDs:LED_0805_HandSoldering" H 6600 1200 50  0001 C CNN
 F 3 "" H 6600 1200 50  0001 C CNN
 	1    6600 1200
@@
 F 0 "D2" H 6600 1600 50  0000 C CNN
 F 1 "LED" H 6600 1400 50  0000 C CNN
-F 2 "" H 6600 1500 50  0001 C CNN
+F 2 "LEDs:LED_0805_HandSoldering" H 6600 1500 50  0001 C CNN
 F 3 "" H 6600 1500 50  0001 C CNN
 	1    6600 1500
@@
 F 0 "D3" H 6600 1900 50  0000 C CNN
 F 1 "LED" H 6600 1700 50  0000 C CNN
-F 2 "" H 6600 1800 50  0001 C CNN
+F 2 "LEDs:LED_0805_HandSoldering" H 6600 1800 50  0001 C CNN
 F 3 "" H 6600 1800 50  0001 C CNN
 	1    6600 1800
@@
 F 0 "R4" V 7130 1200 50  0000 C CNN
 F 1 "R" V 7050 1200 50  0000 C CNN
-F 2 "" V 6980 1200 50  0001 C CNN
+F 2 "Resistors_SMD:R_0805_HandSoldering" V 6980 1200 50  0001 C CNN
 F 3 "" H 7050 1200 50  0001 C CNN
 	1    7050 1200
@@
 F 0 "R5" V 7130 1500 50  0000 C CNN
 F 1 "R" V 7050 1500 50  0000 C CNN
-F 2 "" V 6980 1500 50  0001 C CNN
+F 2 "Resistors_SMD:R_0805_HandSoldering" V 6980 1500 50  0001 C CNN
 F 3 "" H 7050 1500 50  0001 C CNN
 	1    7050 1500
@@
 F 0 "R6" V 7130 1800 50  0000 C CNN
 F 1 "R" V 7050 1800 50  0000 C CNN
-F 2 "" V 6980 1800 50  0001 C CNN
+F 2 "Resistors_SMD:R_0805_HandSoldering" V 6980 1800 50  0001 C CNN
 F 3 "" H 7050 1800 50  0001 C CNN
 	1    7050 1800
@@
 F 0 "J3" H 2600 5450 50  0000 C CNN
 F 1 "Serial" H 2600 4950 50  0000 C CNN
-F 2 "" H 2600 5250 50  0001 C CNN
+F 2 "Pin_Headers:Pin_Header_Straight_1x04_Pitch2.54mm" H 2600 5250 50  0001 C CNN
 F 3 "" H 2600 5250 50  0001 C CNN
 	1    2600 5250
@@
 F 0 "J4" H 2600 6250 50  0000 C CNN
 F 1 "I2C" H 2600 5750 50  0000 C CNN
-F 2 "" H 2600 6050 50  0001 C CNN
+F 2 "Pin_Headers:Pin_Header_Straight_1x04_Pitch2.54mm" H 2600 6050 50  0001 C CNN
 F 3 "" H 2600 6050 50  0001 C CNN
 	1    2600 6050
@@
 F 0 "J7" H 3700 6500 50  0000 C CNN
 F 1 "Conn_01x06" H 3700 5800 50  0000 C CNN
-F 2 "" H 3700 6200 50  0001 C CNN
+F 2 "Pin_Headers:Pin_Header_Straight_1x06_Pitch2.54mm" H 3700 6200 50  0001 C CNN
 F 3 "" H 3700 6200 50  0001 C CNN
 	1    3700 6200
@@
 F 0 "R3" V 7080 3800 50  0000 C CNN
 F 1 "R" V 7000 3800 50  0000 C CNN
-F 2 "" V 6930 3800 50  0001 C CNN
+F 2 "Resistors_SMD:R_0805_HandSoldering" V 6930 3800 50  0001 C CNN
 F 3 "" H 7000 3800 50  0001 C CNN
 	1    7000 3800
@@
 F 0 "J2" H 2400 4100 50  0000 C CNN
 F 1 "Conn_01x02" H 2400 3800 50  0000 C CNN
-F 2 "" H 2400 4000 50  0001 C CNN
+F 2 "Pin_Headers:Pin_Header_Straight_1x02_Pitch2.54mm" H 2400 4000 50  0001 C CNN
 F 3 "" H 2400 4000 50  0001 C CNN
 	1    2400 4000
@@
 F 0 "J6" H 3350 5450 50  0000 C CNN
 F 1 "SoftSerial" H 3350 4950 50  0000 C CNN
-F 2 "" H 3350 5250 50  0001 C CNN
+F 2 "Pin_Headers:Pin_Header_Straight_1x04_Pitch2.54mm" H 3350 5250 50  0001 C CNN
 F 3 "" H 3350 5250 50  0001 C CNN
 	1    3350 5250
@@
 F 0 "J5" H 3350 4100 50  0000 C CNN
 F 1 "Conn_01x02" H 3350 3800 50  0000 C CNN
-F 2 "" H 3350 4000 50  0001 C CNN
+F 2 "Pin_Headers:Pin_Header_Straight_1x02_Pitch2.54mm" H 3350 4000 50  0001 C CNN
 F 3 "" H 3350 4000 50  0001 C CNN
 	1    3350 4000
@@
 F 0 "R1" V 4280 5150 50  0000 C CNN
 F 1 "R" V 4200 5150 50  0000 C CNN
-F 2 "" V 4130 5150 50  0001 C CNN
+F 2 "Resistors_SMD:R_0805_HandSoldering" V 4130 5150 50  0001 C CNN
 F 3 "" H 4200 5150 50  0001 C CNN
 	1    4200 5150
@@
 F 0 "R2" V 4280 5450 50  0000 C CNN
 F 1 "R" V 4200 5450 50  0000 C CNN
-F 2 "" V 4130 5450 50  0001 C CNN
+F 2 "Resistors_SMD:R_0805_HandSoldering" V 4130 5450 50  0001 C CNN
 F 3 "" H 4200 5450 50  0001 C CNN
 	1    4200 5450
@@
 F 0 "SW1" H 6700 4950 50  0000 C CNN
 F 1 "SW_DPST" H 6700 4550 50  0000 C CNN
-F 2 "" H 6700 4750 50  0001 C CNN
+F 2 "def-footprints:Switches_Push_Switch_THD" H 6700 4750 50  0001 C CNN
 F 3 "" H 6700 4750 50  0001 C CNN
 	1    6700 4750
@@
 F 0 "J8" H 4200 4100 50  0000 C CNN
 F 1 "Conn_01x02" H 4200 3800 50  0000 C CNN
-F 2 "" H 4200 4000 50  0001 C CNN
+F 2 "Pin_Headers:Pin_Header_Straight_1x02_Pitch2.54mm" H 4200 4000 50  0001 C CNN
 F 3 "" H 4200 4000 50  0001 C CNN
 	1    4200 4000
@@
 F 0 "JP1" H 8650 1600 50  0000 C CNN
 F 1 "Jumper_NO_Small" H 8660 1640 50  0001 C CNN
-F 2 "" H 8650 1700 50  0001 C CNN
+F 2 "def-footprints:Miscellaneous_Solder_Jumper" H 8650 1700 50  0001 C CNN
 F 3 "" H 8650 1700 50  0001 C CNN
 	1    8650 1700

Commit message: Finished prototype PCB
Parts:
- removed J7: Conn_01x06, Pin_Headers:Pin_Header_Straight_1x06_Pitch2.54mm, symbol Conn_01x06
- removed XA1: Arduino_Micro_Socket, symbol Arduino_Micro_Socket
- added J7: Conn_01x05, Pin_Headers:Pin_Header_Straight_1x05_Pitch2.54mm, symbol Conn_01x05
- added XA1: Arduino_PRO_Micro, def-footprints:Board_Arduino_Pro_Micro, symbol Arduino_PRO_Micro
- U2: footprint (none) -> def-footprints:Board_DC_DC_module_RT8272
Connections:
- net +5V: now also J7.1 (Pin_1), XA1.VCC
- net BUTTON: now also XA1.D4
- net GND: now also J7.5 (Pin_5), XA1.GND
- net IR_IN: now also XA1.A0
- net LED1: now also XA1.D5
- net LED2: now also XA1.D6
- net LED3: now also XA1.D9
- net LED_IR: now also XA1.D10
- net MISO: now also J7.2 (Pin_2), XA1.D14 (D14_SPI_MISO)
- net MOSI: now also J7.3 (Pin_3), XA1.D15 (D15_SPI_SCK)
- net Rx: now also XA1.D0 (D0_RX0)
- net SCK: now also J7.4 (Pin_4), XA1.D16 (D16_SPI_MOSI)
- net SCL: now also XA1.D3 (D3_SCL)
- net SDA: now also XA1.D2 (D2_SDA)
- net SoftRx: now also XA1.D8
- net SoftTx: now also XA1.D7 (D7_INT4)
- net Tx: now also XA1.D1 (D1_TX0)
- net VCC: now also XA1.RAW (VRAW)
- no-connect marks 13 -> 4
Changed lines of the file:
@@
 $EndDescr
-$Comp
-L Arduino_Micro_Socket XA1
-U 1 1 5BD3A6C9
-P 3350 2150
-F 0 "XA1" V 3450 2150 60  0000 C CNN
-F 1 "Arduino_Micro_Socket" V 3250 2150 60  0000 C CNN
-F 2 "" H 5150 5900 60  0001 C CNN
-F 3 "" H 5150 5900 60  0001 C CNN
-	1    3350 2150
-	1    0    0    -1
-$EndComp
 $Comp
 L Conn_01x02 J1
@@
 $EndComp
 $Comp
-L Conn_01x06 J7
-U 1 1 5BD3AB69
-P 3700 6200
-F 0 "J7" H 3700 6500 50  0000 C CNN
-F 1 "Conn_01x06" H 3700 5800 50  0000 C CNN
-F 2 "Pin_Headers:Pin_Header_Straight_1x06_Pitch2.54mm" H 3700 6200 50  0001 C CNN
-F 3 "" H 3700 6200 50  0001 C CNN
-	1    3700 6200
-	1    0    0    -1
-$EndComp
-$Comp
 L CQY99 D4
 U 1 1 5BD3B0B4
@@
 	1    0    0    -1
 $EndComp
-Text Label 5150 2350 2    60   ~ 0
+Text Label 5100 1950 2    60   ~ 0
 MISO
-Text Label 5150 2450 2    60   ~ 0
+Text Label 5100 2050 2    60   ~ 0
 MOSI
-Text Label 5150 2550 2    60   ~ 0
+Text Label 5100 2150 2    60   ~ 0
 SCK
-Text Label 5150 2650 2    60   ~ 0
-SS
 $Comp
 L Conn_01x02 J2
@@
 L +5V #PWR07
 U 1 1 5BD648A4
-P 1500 2950
-F 0 "#PWR07" H 1500 2800 50  0001 C CNN
-F 1 "+5V" H 1500 3090 50  0000 C CNN
-F 2 "" H 1500 2950 50  0001 C CNN
-F 3 "" H 1500 2950 50  0001 C CNN
-	1    1500 2950
+P 1900 2500
+F 0 "#PWR07" H 1900 2350 50  0001 C CNN
+F 1 "+5V" H 1900 2640 50  0000 C CNN
+F 2 "" H 1900 2500 50  0001 C CNN
+F 3 "" H 1900 2500 50  0001 C CNN
+	1    1900 2500
 	1    0    0    -1
 $EndComp
@@
 Text Label 3000 6300 0    60   ~ 0
 SCK
-Text Label 3000 6400 0    60   ~ 0
-SS
 $Comp
 L +5V #PWR016
@@
 L GND #PWR017
 U 1 1 5BD6605E
-P 3000 6500
-F 0 "#PWR017" H 3000 6250 50  0001 C CNN
-F 1 "GND" H 3000 6350 50  0000 C CNN
-F 2 "" H 3000 6500 50  0001 C CNN
-F 3 "" H 3000 6500 50  0001 C CNN
-	1    3000 6500
-	1    0    0    -1
-$EndComp
-Wire Wire Line
-	4650 2350 5150 2350
-Wire Wire Line
-	4650 2450 5150 2450
-Wire Wire Line
-	4650 2550 5150 2550
-Wire Wire Line
-	4650 2650 5150 2650
+P 3000 6400
+F 0 "#PWR017" H 3000 6150 50  0001 C CNN
+F 1 "GND" H 3000 6250 50  0000 C CNN
+F 2 "" H 3000 6400 50  0001 C CNN
+F 3 "" H 3000 6400 50  0001 C CNN
+	1    3000 6400
+	1    0    0    -1
+$EndComp
+Wire Wire Line
+	4650 1950 5100 1950
+Wire Wire Line
+	4650 2050 5100 2050
+Wire Wire Line
+	4650 2150 5100 2150
 Wire Wire Line
 	6750 1200 6900 1200
@@
 	1150 4000 1150 3900
 Wire Wire Line
-	1300 3050 2050 3050
-Wire Wire Line
-	1300 3050 1300 2950
+	1700 2600 2050 2600
+Wire Wire Line
+	1700 2600 1700 2500
 Wire Wire Line
 	7150 2850 7350 2850
@@
 	7350 2850 7350 2750
 Wire Wire Line
-	1500 2950 2050 2950
+	1900 2500 2050 2500
 Wire Wire Line
 	2050 1250 1500 1250
@@
 	3500 6300 3000 6300
 Wire Wire Line
-	3500 6400 3000 6400
-Wire Wire Line
 	3000 6000 3500 6000
 Wire Wire Line
 	3000 6000 3000 5950
 Wire Wire Line
-	3000 6500 3500 6500
+	3000 6400 3500 6400
 Wire Wire Line
 	7150 3050 7450 3050
 Wire Wire Line
-	4650 1950 5100 1950
+	2050 2150 1500 2150
 Text Label 5100 1850 2    60   ~ 0
 LED_IR
-Text Label 5100 1950 2    60   ~ 0
+Text Label 1500 2150 0    60   ~ 0
 IR_IN
 Text Label 7450 3050 2    60   ~ 0
@@
 L GND #PWR020
 U 1 1 5BD667C6
-P 1800 2750
-F 0 "#PWR020" H 1800 2500 50  0001 C CNN
-F 1 "GND" H 1800 2600 50  0000 C CNN
-F 2 "" H 1800 2750 50  0001 C CNN
-F 3 "" H 1800 2750 50  0001 C CNN
-	1    1800 2750
-	1    0    0    -1
-$EndComp
-Wire Wire Line
-	1800 2650 1800 2750
-Wire Wire Line
-	2050 2650 1800 2650
-NoConn ~ 2050 2850
-NoConn ~ 2050 2750
-NoConn ~ 2050 2450
-NoConn ~ 2050 2350
-NoConn ~ 2050 2250
-NoConn ~ 2050 2150
+P 1500 2500
+F 0 "#PWR020" H 1500 2250 50  0001 C CNN
+F 1 "GND" H 1500 2350 50  0000 C CNN
+F 2 "" H 1500 2500 50  0001 C CNN
+F 3 "" H 1500 2500 50  0001 C CNN
+	1    1500 2500
+	1    0    0    -1
+$EndComp
 NoConn ~ 2050 2050
 NoConn ~ 2050 1950
 NoConn ~ 2050 1850
-NoConn ~ 4650 2050
-NoConn ~ 4650 2150
-NoConn ~ 4650 2850
-NoConn ~ 4650 2950
+NoConn ~ 4650 2500
 $Comp
 L R R1
@@
 F 0 "U2" H 9550 1200 60  0000 C CNN
 F 1 "DC_Converter_RT8272" H 9300 1650 60  0000 C CNN
-F 2 "" H 9390 1150 60  0001 C CNN
+F 2 "def-footprints:Board_DC_DC_module_RT8272" H 9390 1150 60  0001 C CNN
 F 3 "" H 9390 1150 60  0001 C CNN
 	1    9350 1400
@@
 L VCC #PWR035
 U 1 1 5BD6AC04
-P 1300 2950
-F 0 "#PWR035" H 1300 2800 50  0001 C CNN
-F 1 "VCC" H 1300 3100 50  0000 C CNN
-F 2 "" H 1300 2950 50  0001 C CNN
-F 3 "" H 1300 2950 50  0001 C CNN
-	1    1300 2950
+P 1700 2500
+F 0 "#PWR035" H 1700 2350 50  0001 C CNN
+F 1 "VCC" H 1700 2650 50  0000 C CNN
+F 2 "" H 1700 2500 50  0001 C CNN
+F 3 "" H 1700 2500 50  0001 C CNN
+	1    1700 2500
 	1    0    0    -1
 $EndComp
 Text Notes 3000 4450 0    60   ~ 0
 Extra Power
+Wire Wire Line
+	2050 2400 2050 2250
+Wire Wire Line
+	1500 2500 1500 2250
+Wire Wire Line
+	1500 2250 2050 2250
+$Comp
+L Conn_01x05 J7
+U 1 1 5BD78FCB
+P 3700 6200
+F 0 "J7" H 3700 6500 50  0000 C CNN
+F 1 "Conn_01x05" H 3700 5900 50  0000 C CNN
+F 2 "Pin_Headers:Pin_Header_Straight_1x05_Pitch2.54mm" H 3700 6200 50  0001 C CNN
+F 3 "" H 3700 6200 50  0001 C CNN
+	1    3700 6200
+	1    0    0    -1
+$EndComp
+$Comp
+L Arduino_PRO_Micro XA1
+U 1 1 5BD7A9B9
+P 3350 2150
+F 0 "XA1" H 3200 3100 60  0000 C CNN
+F 1 "Arduino_PRO_Micro" H 3400 1650 60  0000 C CNN
+F 2 "def-footprints:Board_Arduino_Pro_Micro" H 5150 5900 60  0001 C CNN
+F 3 "" H 5150 5900 60  0001 C CNN
+	1    3350 2150
+	1    0    0    -1
+$EndComp
 $EndSCHEMATC
