File: hardware/project-x.kicad_pcb (KiCad board)
At the start: 2 copper layers, 0 parts

Commit message: Start basic layout
Parts:
- added D1: LED, LEDs:LED_0805_HandSoldering, F.Cu at (172.7, 129.5)
- added D2: LED, LEDs:LED_0805_HandSoldering, F.Cu at (172.7, 132.1)
- added D3: LED, LEDs:LED_0805_HandSoldering, F.Cu at (172.7, 134.6)
- added D4: CQY99, LEDs:LED_D5.0mm, F.Cu at (139.7, 58.4)
- added J1: Conn_01x02, Pin_Headers:Pin_Header_Straight_1x02_Pitch2.54mm, F.Cu at (231.3, 131.9)
- added J2: Conn_01x02, Pin_Headers:Pin_Header_Straight_1x02_Pitch2.54mm, F.Cu at (219.7, 140.7)
- added J3: Serial, Pin_Headers:Pin_Header_Straight_1x04_Pitch2.54mm, F.Cu at (204.9, 136.2)
- added J4: I2C, Pin_Headers:Pin_Header_Straight_1x04_Pitch2.54mm, F.Cu at (235.0, 117.6)
- added J5: Conn_01x02, Pin_Headers:Pin_Header_Straight_1x02_Pitch2.54mm, F.Cu at (241.8, 117.6)
- added J6: SoftSerial, Pin_Headers:Pin_Header_Straight_1x04_Pitch2.54mm, F.Cu at (211.1, 136.2)
- added J7: Conn_01x06, Pin_Headers:Pin_Header_Straight_1x06_Pitch2.54mm, F.Cu at (197.8, 124.0)
- added J8: Conn_01x02, Pin_Headers:Pin_Header_Straight_1x02_Pitch2.54mm, F.Cu at (221.8, 131.5)
- added JP1: Jumper_NO_Small, def-footprints:Miscellaneous_Solder_Jumper, F.Cu at (227.6, 115.0)
- added R1: R, Resistors_SMD:R_0805_HandSoldering, F.Cu at (228.6, 121.9)
- added R2: R, Resistors_SMD:R_0805_HandSoldering, F.Cu at (249.1, 117.0)
- added R3: R, Resistors_SMD:R_0805_HandSoldering, F.Cu at (239.6, 126.2)
- added R4: R, Resistors_SMD:R_0805_HandSoldering, F.Cu at (227.1, 146.1)
- added R5: R, Resistors_SMD:R_0805_HandSoldering, F.Cu at (244.7, 126.2)
- added R6: R, Resistors_SMD:R_0805_HandSoldering, F.Cu at (238.6, 131.7)
- added REF***: KiCad-Logo_6mm_SilkScreen, Symbols:KiCad-Logo_6mm_SilkScreen, F.Cu at (111.8, 134.6)
- added SW1: SW_DPST, def-footprints:Switches_Push_Switch_THD, F.Cu at (111.8, 127.0)
- added U1: TSOP382xx, Opto-Devices:IRReceiver_Vishay_MINICAST-3pin, F.Cu at (139.7, 134.6)
Other:
- board outline added: 80 x 94.5 mm

Commit message: Add ASROB logo
Parts:
- added G***: LOGO, def-footprints:Logo_ASROB_2.5x2.5_cm, B.Cu at (142.6, 95.5)

Commit message: Finished prototype PCB
Parts:
- added REF**: MountingHole_5.5mm, Mounting_Holes:MountingHole_5.5mm, F.Cu at (169.3, 120.6)
- added REF**: MountingHole_3mm, Mounting_Holes:MountingHole_3mm, F.Cu at (174.1, 147.6)
- added REF**: MountingHole_3mm, Mounting_Holes:MountingHole_3mm, F.Cu at (108.1, 147.6)
- added REF**: MountingHole_3mm, Mounting_Holes:MountingHole_3mm, F.Cu at (165.1, 59.6)
- added REF**: MountingHole_3mm, Mounting_Holes:MountingHole_3mm, F.Cu at (117.1, 59.6)
- added REF**: MountingHole_5.5mm, Mounting_Holes:MountingHole_5.5mm, F.Cu at (112.8, 120.6)
- added REF***: OSHW-Logo_5.7x6mm_SilkScreen, Symbols:OSHW-Logo_5.7x6mm_SilkScreen, F.Cu at (108.9, 96.9)
- added U2: DC_Converter_RT8272, def-footprints:Board_DC_DC_module_RT8272, F.Cu at (165.9, 111.8)
- added XA1: Arduino_PRO_Micro, def-footprints:Board_Arduino_Pro_Micro, F.Cu at (119.4, 118.6)
- J7: value Conn_01x06 -> Conn_01x05; footprint Pin_Headers:Pin_Header_Straight_1x06_Pitch2.54mm -> Pin_Headers:Pin_Header_Straight_1x05_Pitch2.54mm
- moved J2 125.5 mm to (125.5, 57.9), turned to 90 degrees
- moved J8 117.7 mm to (107.2, 104.6), turned to 90 degrees
- moved R3 116.9 mm to (141.2, 63.0)
- moved J5 106.4 mm to (153.7, 57.9), turned to 90 degrees
- moved R2 93.5 mm to (156.2, 127.8), turned to 90 degrees
- moved J6 87.1 mm to (131.3, 101.3), turned to 270 degrees
- moved J1 85.5 mm to (150.9, 102.9)
- moved J4 85.2 mm to (151.1, 132.6), turned to 90 degrees
- moved R5 78.1 mm to (166.9, 132.1)
- moved J3 76.2 mm to (128.8, 131.8), turned to 270 degrees
- moved R1 75.2 mm to (153.7, 127.8), turned to 90 degrees
- moved R6 71.8 mm to (166.9, 134.6)
- moved R4 62.4 mm to (166.9, 129.5)
- moved JP1 57.2 mm to (172.5, 99.8)
- moved J7 51.2 mm to (148.1, 111.8)
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Connections:
- J7 pad 5: /SS -> GND
Routing:
- net VCC: track 0.00 -> 68.8 mm
- net +5V: track 0.00 -> 54.9 mm, vias 0 -> 4
- net /SCL: track 0.00 -> 53.7 mm
- net /LED_IR: track 0.00 -> 51.5 mm, vias 0 -> 2
- net /SDA: track 0.00 -> 51.1 mm
- net /LED1: track 0.00 -> 48.8 mm
- net /LED2: track 0.00 -> 47.0 mm
- net /LED3: track 0.00 -> 39.5 mm
- net /IR_IN: track 0.00 -> 29.9 mm, vias 0 -> 2
- net +BATT: track 0.00 -> 26.3 mm
- net /SoftRx: track 0.00 -> 26.0 mm, vias 0 -> 2
- net /SoftTx: track 0.00 -> 25.6 mm, vias 0 -> 2
- net /MOSI: track 0.00 -> 24.7 mm
- net /MISO: track 0.00 -> 22.3 mm
- net /SCK: track 0.00 -> 22.1 mm, vias 0 -> 2
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- added copper zone on F.Cu, net +5V
- added copper zone on B.Cu, net GND
Other:
- board size 80 x 94.5 mm -> 76 x 96.1 mm
- net class pwr added: clearance 0.2, trace_width 0.55, via_dia 0.6, via_drill 0.4
- board text added: "+"
- board text added: "-"
- board text added: "BAT IN 2S-3S"
- board text added: "CAM"
- board text added: "CAR PWR"
- board text added: "GND"
- board text added: "I2C"
- board text added: "MISO"
- board text added: "MOSI"
- board text added: "PWR"
- board text added: "RX"
- board text added: "SCK"
- board text added: "SCL"
- board text added: "SDA"
- board text added: "SERIAL"
- board text added: "SOFT"
- board text added: "SPI"
- board text added: "TX"
- board text added: "VCC"

Commit message: Add author, url, version to silkcreen
Parts:
- added G***: LOGO, def-footprints:Logo_Project_X, B.Cu at (141.1, 94.6)
- moved G*** 2.20 mm to (140.4, 77.3)
Other:
- board text added: "David Estevez Fernandez"
- board text added: "github.com/asrob-uc3m/project-x"
- board text added: "v0.1"

Commit message: Relocate ASROB logo
Parts:
- moved G*** 0.81 mm to (140.3, 76.5)
Changed lines of the file:
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@@
   )
   (module def-footprints:Logo_ASROB_2.5x2.5_cm (layer B.Cu)
-    (at 140.4 77.3 180)
+    (at 140.3 76.5 180)
     (fp_text reference G*** (at 0 0 180) (layer B.SilkS) hide
       (effects (font (thickness 0.3)) (justify mirror))
